Commit message: update

File: ros2_ws/install/zed_multi_camera/share/zed_multi_camera/urdf/zed_multi.urdf.xacro (robot description, xacro)
@@ -1,59 +1 @@
-<?xml version="1.0"?>
-<!--
-// Copyright 2022 Stereolabs
-//
-// Licensed under the Apache License, Version 2.0 (the "License");
-// you may not use this file except in compliance with the License.
-// You may obtain a copy of the License at
-//
-//      http://www.apache.org/licenses/LICENSE-2.0
-//
-// Unless required by applicable law or agreed to in writing, software
-// distributed under the License is distributed on an "AS IS" BASIS,
-// WITHOUT WARRANTIES OR CONDITIONS OF ANY KIND, either express or implied.
-// See the License for the specific language governing permissions and
-// limitations under the License.
--->
-<!-- *** THIS IS AN EXAMPLE FILE FOR A MULTI-CAMERA CONFIGURATION *** -->
-<!--
-  This xacro file allows to configure a multi-camera system with two cameras
-  mounted on a plate, distant 12 cm and looking at opposite directions.
-  It demonstrates how to configure the URDF/xacro file to create a working
-  multi-camera rig.
--->
-<!--
-    ___                        ___
-    | |                        | |
-    |_|                        |_|
-    _|____________*_____________|_
-    ______________*_______________
-                  |
-    +6cm          0            -6cm
- zed_front  zed_multi_link    zed_back
--->
-<robot name="zed_multi_camera" xmlns:xacro="http://ros.org/wiki/xacro">
-  <xacro:property name="M_PI"     value="3.1415926535897931" />
-  <!-- Define the required parameters -->
-  <xacro:arg name="multi_link" default="zed_multi_link" />
-  <xacro:arg name="camera_name_0" default="zed_front" />
-  <xacro:arg name="camera_name_1" default="zed_rear" />
-  <!-- Define the reference links -->
-  <link name="$(arg multi_link)" />
-  <link name="$(arg camera_name_0)_camera_link" />
-  <link name="$(arg camera_name_1)_camera_link" />
-  <!-- Note the URDF of the cameras are loaded by the respective launch files.
-       We must only provide the position of each of them with respect to the reference link -->
-  <!-- Define the position of the front camera with respect to the reference link -->
-  <joint name="$(arg camera_name_0)_camera_joint" type="fixed">
-      <parent link="$(arg camera_name_0)_camera_link"/>
-      <child link="$(arg multi_link)"/>
-      <origin xyz="0.06 0.0 0.0" rpy="0 0 0" />
-  </joint>
-  <!-- Define the position of the rear camera with respect to the reference link -->
-  <joint name="$(arg camera_name_1)_camera_joint" type="fixed">
-      <parent link="$(arg multi_link)"/>
-      <child link="$(arg camera_name_1)_camera_link"/>
-      <origin xyz="-0.06 0.0 0.0" rpy="0 0 ${M_PI}" />
-  </joint>
-  <!-- NOTE: Replicate the same XML code above for all the cameras of the multi-camera system if more cameras are used -->
-</robot>
+/home/aiv/YongJun_ws/ros2_ws/src/zed-ros2-examples/tutorials/zed_multi_camera/urdf/zed_multi.urdf.xacro

File: ros2_ws/install/zed_robot_integration/share/zed_robot_integration/urdf/zed_robot_dual.urdf.xacro (robot description, xacro)
@@ -1,64 +1 @@
-<?xml version="1.0"?>
-<!--
-// Copyright 2024 Stereolabs
-//
-// Licensed under the Apache License, Version 2.0 (the "License");
-// you may not use this file except in compliance with the License.
-// You may obtain a copy of the License at
-//
-//      http://www.apache.org/licenses/LICENSE-2.0
-//
-// Unless required by applicable law or agreed to in writing, software
-// distributed under the License is distributed on an "AS IS" BASIS,
-// WITHOUT WARRANTIES OR CONDITIONS OF ANY KIND, either express or implied.
-// See the License for the specific language governing permissions and
-// limitations under the License.
--->
-<robot name="zedbot_scoutm" xmlns:xacro="http://ros.org/wiki/xacro">
-  <xacro:arg name="camera_name_1"   default="zed_front" />
-  <xacro:arg name="camera_name_2"   default="zed_back" />
-  <xacro:arg name="camera_model_1"  default="zedx" />
-  <xacro:arg name="camera_model_2"  default="zedx" />
-  <xacro:arg name="use_zed_localization" default="true" />
-  <xacro:property name="M_PI"     value="3.1415926535897931" />
-  <!-- Include the robot (AgileX Scout mini) -->
-  <xacro:include filename="$(find scout_description)/urdf/scout_mini.xacro" />
-  <!-- Load the ZED xacro macro -->
-  <xacro:include filename="$(find zed_wrapper)/urdf/zed_macro.urdf.xacro" />
-  <!-- Add the first ZED Camera -->
-  <xacro:zed_camera name="$(arg camera_name_1)" model="$(arg camera_model_1)" />
-  <!-- Add the second ZED Camera -->
-  <xacro:zed_camera name="$(arg camera_name_2)" model="$(arg camera_model_2)" />
-  <!-- Add the joints to connect the ZED Cameras to the robot -->
-  <xacro:if value="$(arg use_zed_localization)">
-    <!-- ZED Localization -> The reference link is '$(arg camera_name_1)_camera_link' and 'base_link' is a child -->
-    <joint name="$(arg camera_name_1)_joint" type="fixed">
-      <parent link="$(arg camera_name_1)_camera_link"/>
-      <child link="base_link"/>
-      <origin
-        xyz="-0.12 0.0 -0.25"
-        rpy="0 0 0"
-      />
-    </joint>
-  </xacro:if>
-  <xacro:unless value="$(arg use_zed_localization)">
-    <!-- NO ZED Localization -> '$(arg camera_name)_camera_link' is a child of 'base_link' -->
-    <joint name="$(arg camera_name_1)_joint" type="fixed">
-      <parent link="base_link"/>
-      <child link="$(arg camera_name_1)_camera_link"/>
-      <origin
-        xyz="0.12 0.0 0.25"
-        rpy="0 0 0"
-      />
-    </joint>
-  </xacro:unless>
-  <!-- Add the joint of the second camera -->
-  <joint name="$(arg camera_name_2)_joint" type="fixed">
-    <parent link="base_link"/>
-    <child link="$(arg camera_name_2)_camera_link"/>
-    <origin
-      xyz="-0.12 0.0 0.25"
-      rpy="0 0 ${M_PI}"
-    />
-  </joint>
-</robot>
+/home/aiv/YongJun_ws/ros2_ws/src/zed-ros2-examples/tutorials/zed_robot_integration/urdf/zed_robot_dual.urdf.xacro

File: ros2_ws/install/zed_robot_integration/share/zed_robot_integration/urdf/zed_robot_mono.urdf.xacro (robot description, xacro)
@@ -1,50 +1 @@
-<?xml version="1.0"?>
-<!--
-// Copyright 2024 Stereolabs
-//
-// Licensed under the Apache License, Version 2.0 (the "License");
-// you may not use this file except in compliance with the License.
-// You may obtain a copy of the License at
-//
-//      http://www.apache.org/licenses/LICENSE-2.0
-//
-// Unless required by applicable law or agreed to in writing, software
-// distributed under the License is distributed on an "AS IS" BASIS,
-// WITHOUT WARRANTIES OR CONDITIONS OF ANY KIND, either express or implied.
-// See the License for the specific language governing permissions and
-// limitations under the License.
--->
-<robot name="zedbot_scoutm" xmlns:xacro="http://ros.org/wiki/xacro">
-  <xacro:arg name="camera_name"   default="zed" />
-  <xacro:arg name="camera_model"  default="zedx" />
-  <xacro:arg name="use_zed_localization" default="true" />
-  <xacro:arg name="baseline" default="0.0" />
-  <!-- Include the robot (e.g. AgileX Scout mini) -->
-  <xacro:include filename="$(find scout_description)/urdf/scout_mini.xacro" />
-  <!-- Add one ZED Camera -->
-  <xacro:include filename="$(find zed_wrapper)/urdf/zed_macro.urdf.xacro" />
-  <xacro:zed_camera name="$(arg camera_name)" model="$(arg camera_model)" baseline="$(arg baseline)"/>
-  <!-- Add a joint to connect the ZED Camera to the robot -->
-  <xacro:if value="$(arg use_zed_localization)">
-    <!-- ZED Localization -> The reference link is '$(arg camera_name)_camera_link' and 'base_link' is a child -->
-    <joint name="$(arg camera_name)_joint" type="fixed">
-      <parent link="$(arg camera_name)_camera_link"/>
-      <child link="base_link"/>
-      <origin
-        xyz="-0.12 0.0 -0.25"
-        rpy="0 0 0"
-      />
-    </joint>
-  </xacro:if>
-  <xacro:unless value="$(arg use_zed_localization)">
-    <!-- NO ZED Localization -> '$(arg camera_name)_camera_link' is a child of 'base_link' -->
-    <joint name="$(arg camera_name)_joint" type="fixed">
-      <parent link="base_link"/>
-      <child link="$(arg camera_name)_camera_link"/>
-      <origin
-        xyz="0.12 0.0 0.25"
-        rpy="0 0 0"
-      />
-    </joint>
-  </xacro:unless>
-</robot>
+/home/aiv/YongJun_ws/ros2_ws/src/zed-ros2-examples/tutorials/zed_robot_integration/urdf/zed_robot_mono.urdf.xacro

File: ros2_ws/install/zed_wrapper/share/zed_wrapper/urdf/include/materials.urdf.xacro (robot description, xacro)
@@ -1,39 +1 @@
-<?xml version="1.0"?>
-<!--
-// Copyright 2022 Stereolabs
-//
-// Licensed under the Apache License, Version 2.0 (the "License");
-// you may not use this file except in compliance with the License.
-// You may obtain a copy of the License at
-//
-//      http://www.apache.org/licenses/LICENSE-2.0
-//
-// Unless required by applicable law or agreed to in writing, software
-// distributed under the License is distributed on an "AS IS" BASIS,
-// WITHOUT WARRANTIES OR CONDITIONS OF ANY KIND, either express or implied.
-// See the License for the specific language governing permissions and
-// limitations under the License.
--->
-<robot>
-    <material name="zed_mat">
-        <color rgba="0.8 0.8 0.8 1.0"/>
-    </material>
-    <material name="zedm_mat">
-        <color rgba="0 0 0 1.0"/>
-    </material>
-    <material name="zed2_mat">
-        <color rgba="0.25 0.25 0.25 1.0"/>
-    </material>
-    <material name="zed2i_mat">
-        <color rgba="0.25 0.25 0.25 1.0"/>
-    </material>
-    <material name="zedx_mat">
-        <color rgba="0.25 0.25 0.25 1.0"/>
-    </material>
-    <material name="zedxm_mat">
-        <color rgba="0.25 0.25 0.25 1.0"/>
-    </material>
-    <material name="virtual_mat">
-        <color rgba="0.25 0.25 0.25 1.0"/>
-    </material>
-</robot>
+/home/aiv/YongJun_ws/ros2_ws/src/zed-ros2-wrapper/zed_wrapper/urdf/include/materials.urdf.xacro

File: ros2_ws/install/zed_wrapper/share/zed_wrapper/urdf/zed_descr.urdf.xacro (robot description, xacro)
@@ -1,30 +1 @@
-<?xml version="1.0"?>
-<!--
-// Copyright 2022 Stereolabs
-//
-// Licensed under the Apache License, Version 2.0 (the "License");
-// you may not use this file except in compliance with the License.
-// You may obtain a copy of the License at
-//
-//      http://www.apache.org/licenses/LICENSE-2.0
-//
-// Unless required by applicable law or agreed to in writing, software
-// distributed under the License is distributed on an "AS IS" BASIS,
-// WITHOUT WARRANTIES OR CONDITIONS OF ANY KIND, either express or implied.
-// See the License for the specific language governing permissions and
-// limitations under the License.
--->
-<robot name="stereolabs_camera" xmlns:xacro="http://ros.org/wiki/xacro">
-  <xacro:arg name="camera_name"   default="zed" />
-  <xacro:arg name="camera_model"  default="zed" />
-  <xacro:arg name="custom_baseline"  default="0.0" />
-  <!-- If GNSS fusion is enabled the position of the antenna with respect to the camera mount point is required -->
-  <xacro:arg name="enable_gnss"   default="false" />
-  <xacro:arg name="gnss_x" default="0.0" />
-  <xacro:arg name="gnss_y" default="0.0" />
-  <xacro:arg name="gnss_z" default="0.0" />
-  <xacro:include filename="$(find zed_wrapper)/urdf/zed_macro.urdf.xacro" />
-  <xacro:zed_camera name="$(arg camera_name)" model="$(arg camera_model)" custom_baseline="$(arg custom_baseline)" enable_gnss="$(arg enable_gnss)">
-	    <origin xyz="$(arg gnss_x) $(arg gnss_y) $(arg gnss_z)" rpy="0 0 0"/>
-  </xacro:zed_camera>
-</robot>
+/home/aiv/YongJun_ws/ros2_ws/src/zed-ros2-wrapper/zed_wrapper/urdf/zed_descr.urdf.xacro

File: ros2_ws/install/zed_wrapper/share/zed_wrapper/urdf/zed_macro.urdf.xacro (robot description, xacro)
@@ -1,202 +1 @@
-<?xml version="1.0"?>
-<!--
-// Copyright 2022 Stereolabs
-//
-// Licensed under the Apache License, Version 2.0 (the "License");
-// you may not use this file except in compliance with the License.
-// You may obtain a copy of the License at
-//
-//      http://www.apache.org/licenses/LICENSE-2.0
-//
-// Unless required by applicable law or agreed to in writing, software
-// distributed under the License is distributed on an "AS IS" BASIS,
-// WITHOUT WARRANTIES OR CONDITIONS OF ANY KIND, either express or implied.
-// See the License for the specific language governing permissions and
-// limitations under the License.
--->
-<robot xmlns:xacro="http://wiki.ros.org/xacro">
-  <xacro:include filename="$(find zed_wrapper)/urdf/include/materials.urdf.xacro" />
-  <xacro:property name="M_PI"     value="3.1415926535897931" />
-  <!--
-    Parameters:
-      - name: the camera's name.  should match the parameter sent to the launch file for this camera
-      - model: the type of camera, one of zed, zedm, zed2, zed2i, zedx, zedxm, virtual
-      - enable_gnss: if true enable the URDF link
-  -->
-  <xacro:macro name="zed_camera" params="name=zed model=zed enable_gnss=false custom_baseline=0 *gnss_origin">
-    <xacro:if value="${model == 'zed'}">
-      <xacro:property name="baseline" value="0.12" />
-      <xacro:property name="height" value="0.03" />
-      <xacro:property name="bottom_slope" value="0.05" />
-      <xacro:property name="screw_offset_x" value="0.0" />
-      <xacro:property name="screw_offset_z" value="0.0" />
-      <xacro:property name="optical_offset_x" value="-0.01" />
-    </xacro:if>
-    <xacro:if value="${model == 'zedm'}">
-      <xacro:property name="baseline" value="0.06" />
-      <xacro:property name="height" value="0.0265" />
-      <xacro:property name="bottom_slope" value="0.0" />
-      <xacro:property name="screw_offset_x" value="0.0" />
-      <xacro:property name="screw_offset_z" value="0.0" />
-      <xacro:property name="optical_offset_x" value="0.0" />
-    </xacro:if>
-    <xacro:if value="${model == 'zed2'}">
-      <xacro:property name="baseline" value="0.12" />
-      <xacro:property name="height" value="0.03" />
-      <xacro:property name="bottom_slope" value="0.05" />
-      <xacro:property name="screw_offset_x" value="0.0" />
-      <xacro:property name="screw_offset_z" value="0.0" />
-      <xacro:property name="optical_offset_x" value="-0.01" />
-    </xacro:if>
-    <xacro:if value="${model == 'zed2i'}">
-      <xacro:property name="baseline" value="0.12" />
-      <xacro:property name="height" value="0.03" />
-      <xacro:property name="bottom_slope" value="0.0" />
-      <xacro:property name="screw_offset_x" value="-0.01" />
-      <xacro:property name="screw_offset_z" value="0.0" />
-      <xacro:property name="optical_offset_x" value="-0.01" />
-    </xacro:if>
-    <xacro:if value="${model == 'zedx'}">
-      <xacro:property name="baseline" value="0.12" />
-      <xacro:property name="height" value="0.032" />
-      <xacro:property name="bottom_slope" value="0.0" />
-      <xacro:property name="screw_offset_x" value="0.0" />
-      <xacro:property name="screw_offset_z" value="-0.016" />
-      <xacro:property name="optical_offset_x" value="-0.01" />
-    </xacro:if>
-    <xacro:if value="${model == 'zedxm'}">
-      <xacro:property name="baseline" value="0.05" />
-      <xacro:property name="height" value="0.032" />
-      <xacro:property name="bottom_slope" value="0.0" />
-      <xacro:property name="screw_offset_x" value="0.0" />
-      <xacro:property name="screw_offset_z" value="-0.016" />
-      <xacro:property name="optical_offset_x" value="-0.01" />
-    </xacro:if>
-    <xacro:if value="${model == 'virtual'}">
-      <xacro:property name="baseline" value="${custom_baseline}" />
-      <xacro:property name="height" value="0.031" />
-      <xacro:property name="bottom_slope" value="0.0" />
-      <xacro:property name="screw_offset_x" value="0.00" />
-      <xacro:property name="screw_offset_z" value="-0.0155" />
-      <xacro:property name="optical_offset_x" value="0.0" />
-    </xacro:if>
-    <!-- Camera mounting point (the threaded screw hole in the bottom) -->
-    <link name="${name}_camera_link" />
-    <!-- Camera Center -->
-    <link name="${name}_camera_center">
-      <xacro:unless value="${model == 'virtual'}">
-        <visual>
-          <origin xyz="${screw_offset_x} 0 ${screw_offset_z}" rpy="0 0 0"/>
-          <geometry>
-            <mesh filename="package://zed_interfaces/meshes/${model}.stl" />
-          </geometry>
-          <material name="${model}_mat" />
-        </visual>
-        <collision>
-          <origin xyz="${screw_offset_x} 0 ${screw_offset_z}" rpy="0 0 0"/>
-          <geometry>
-            <mesh filename="package://zed_interfaces/meshes/${model}.stl" />
-          </geometry>
-        </collision>
-      </xacro:unless>
-    </link>
-    <joint name="${name}_camera_center_joint" type="fixed">
-      <parent link="${name}_camera_link"/>
-      <child link="${name}_camera_center"/>
-      <origin xyz="0 0 ${height/2}" rpy="0 ${bottom_slope} 0" />
-    </joint>
-    <!-- Left Camera -->
-    <link name="${name}_left_camera_frame">
-      <xacro:if value="${model == 'virtual'}">
-        <visual>
-          <origin xyz="0 0 0" rpy="0 0 0"/>
-          <geometry>
-            <mesh filename="package://zed_interfaces/meshes/${model}.stl" />
-          </geometry>
-          <material name="${model}_mat" />
-        </visual>
-        <collision>
-          <origin xyz="0 0 0" rpy="0 0 0"/>
-          <geometry>
-            <mesh filename="package://zed_interfaces/meshes/${model}.stl" />
-          </geometry>
-        </collision>
-      </xacro:if>
-    </link>
-    <joint name="${name}_left_camera_joint" type="fixed">
-      <parent link="${name}_camera_center"/>
-      <child link="${name}_left_camera_frame"/>
-      <origin xyz="${optical_offset_x} ${baseline/2} 0" rpy="0 0 0" />
-    </joint>
-    <link name="${name}_left_camera_optical_frame"/>
-    <joint name="${name}_left_camera_optical_joint" type="fixed">
-      <origin xyz="0 0 0" rpy="-${M_PI/2} 0.0 -${M_PI/2}"/>
-      <parent link="${name}_left_camera_frame"/>
-      <child link="${name}_left_camera_optical_frame"/>
-    </joint>
-    <!-- Right Camera -->
-    <link name="${name}_right_camera_frame">
-      <xacro:if value="${model == 'virtual'}">
-        <visual>
-          <origin xyz="0 0 0" rpy="0 0 0"/>
-          <geometry>
-            <mesh filename="package://zed_interfaces/meshes/${model}.stl" />
-          </geometry>
-          <material name="${model}_mat" />
-        </visual>
-        <collision>
-          <origin xyz="0 0 0" rpy="0 0 0"/>
-          <geometry>
-            <mesh filename="package://zed_interfaces/meshes/${model}.stl" />
-          </geometry>
-        </collision>
-      </xacro:if>
-    </link>
-    <joint name="${name}_right_camera_joint" type="fixed">
-      <parent link="${name}_camera_center"/>
-      <child link="${name}_right_camera_frame"/>
-      <origin xyz="${optical_offset_x} -${baseline/2} 0" rpy="0 0 0" />
-    </joint>
-    <link name="${name}_right_camera_optical_frame"/>
-    <joint name="${name}_right_camera_optical_joint" type="fixed">
-      <origin xyz="0 0 0" rpy="-${M_PI/2} 0.0 -${M_PI/2}"/>
-      <parent link="${name}_right_camera_frame"/>
-      <child link="${name}_right_camera_optical_frame"/>
-    </joint>
-    <!-- ZED2 Sensors -->
-    <xacro:if value="${model == 'zed2'}">
-      <link name="${name}_mag_link" />
-      <joint name="${name}_mag_joint" type="fixed">
-        <parent link="${name}_camera_center"/>
-        <child link="${name}_mag_link"/>
-        <origin xyz="0 0 0" rpy="0 0 0" />
-      </joint>
-      <link name="${name}_baro_link" />
-      <joint name="${name}_baro_joint" type="fixed">
-        <parent link="${name}_camera_center"/>
-        <child link="${name}_baro_link"/>
-        <origin xyz="0 0 0" rpy="0 0 0" />
-      </joint>
-      <link name="${name}_temp_left_link" />
-      <joint name="${name}_temp_left_joint" type="fixed">
-        <parent link="${name}_left_camera_frame"/>
-        <child link="${name}_temp_left_link"/>
-        <origin xyz="0 0 0" rpy="0 0 0" />
-      </joint>
-      <link name="${name}_temp_right_link" />
-      <joint name="${name}_temp_right_joint" type="fixed">
-        <parent link="${name}_right_camera_frame"/>
-        <child link="${name}_temp_right_link"/>
-        <origin xyz="0 0 0" rpy="0 0 0" />
-      </joint>
-    </xacro:if>
-    <xacro:if value="${enable_gnss}">
-      <link name="${name}_gnss_link" />
-      <joint name="${name}_gnss_joint" type="fixed">
-        <parent link="${name}_camera_link"/>
-        <child link="${name}_gnss_link"/>
-        <xacro:insert_block name="gnss_origin" />
-      </joint>
-    </xacro:if>
-  </xacro:macro>
-</robot>
+/home/aiv/YongJun_ws/ros2_ws/src/zed-ros2-wrapper/zed_wrapper/urdf/zed_macro.urdf.xacro
